Commit message: "trying to add thrusters to model"

File: thruster_test.sdf.xacro (robot description, xacro)
@@ -2,14 +2,26 @@
 <sdf version='1.7'>
   <model name='rov_starting_point'>
+  <xacro:macro name="thruster_macro" params="
+        namespace
+        thruster_id
+        *origin">
+        <joint name="${namespace}/thruster_${thruster_id}_joint" type="continuous">
+            <xacro:insert_block name="origin"/>
+            <axis xyz="1 0 0"/>
+            <parent link="${namespace}/box_body"/>
+            <child link="${namespace}/thruster_${thruster_id}"/>
+        </joint>
+        <link name="${namespace}/thruster_${thruster_id}"/>
+    </xacro:macro>
     <link name='box_body'>
       <inertial>
-        <mass>m_box</mass>
+        <mass>4</mass>
         <inertia>
-          <ixx>I_x</ixx>
+          <ixx>4.333333333333333</ixx>
           <ixy>0</ixy>
           <ixz>0</ixz>
-          <iyy>I_y</iyy>
+          <iyy>3.333333333333333</iyy>
           <iyz>0</iyz>
-          <izz>I_z</izz>
+          <izz>1.6666666666666665</izz>
         </inertia>
         <pose>0 0 0 0 -0 0</pose>
@@ -18,10 +30,10 @@
       <enable_wind>0</enable_wind>
       <kinematic>0</kinematic>
-      <pose>0 0 p_z 0 -0 0</pose>
+      <pose>0 0 -1.5 0 -0 0</pose>
       <gravity>1</gravity>
       <visual name='visual'>
         <geometry>
           <box>
-            <size>w_box l_box h_box</size>
+            <size>1 2 3</size>
           </box>
         </geometry>
@@ -49,5 +61,5 @@
         <geometry>
           <box>
-            <size>w_box l_box h_box</size>
+            <size>1 2 3</size>
           </box>
         </geometry>
@@ -112,5 +124,5 @@
         <pose>0 0 0 0 -0 0</pose>
       </inertial>
-      <pose>-0 p_side_y p_z 1.57081 1.57079 1.57081</pose>
+      <pose>-0 1.039 -1.5 1.57081 1.57079 1.57081</pose>
       <gravity>1</gravity>
       <self_collide>0</self_collide>
@@ -121,6 +133,6 @@
         <geometry>
           <cylinder>
-            <radius>r_thruster</radius>
-            <length>l_thruster</length>
+            <radius>0.039</radius>
+            <length>0.112</length>
           </cylinder>
         </geometry>
@@ -148,6 +160,6 @@
         <geometry>
           <cylinder>
-            <radius>r_thruster</radius>
-            <length>l_thruster</length>
+            <radius>0.039</radius>
+            <length>0.112</length>
           </cylinder>
         </geometry>
@@ -212,5 +224,5 @@
         <pose>0 0 0 0 -0 0</pose>
       </inertial>
-      <pose>-0 -p_side_y p_z 1.5708 1.57078 1.5708</pose>
+      <pose>-0 -1.039 -1.5 1.5708 1.57078 1.5708</pose>
       <gravity>1</gravity>
       <self_collide>0</self_collide>
@@ -221,6 +233,6 @@
         <geometry>
           <cylinder>
-            <radius>r_thruster</radius>
-            <length>l_thruster</length>
+            <radius>0.039</radius>
+            <length>0.112</length>
           </cylinder>
         </geometry>
@@ -248,6 +260,6 @@
         <geometry>
           <cylinder>
-            <radius>r_thruster</radius>
-            <length>l_thruster</length>
+            <radius>0.039</radius>
+            <length>0.112</length>
           </cylinder>
         </geometry>
@@ -312,5 +324,5 @@
         <pose>0 0 0 0 -0 0</pose>
       </inertial>
-      <pose>p_up_x p_up_y p_z 0 -0 0</pose>
+      <pose>0.539 0.961 -1.5 0 -0 0</pose>
       <gravity>1</gravity>
       <self_collide>0</self_collide>
@@ -321,6 +333,6 @@
         <geometry>
           <cylinder>
-            <radius>r_thruster</radius>
-            <length>l_thruster</length>
+            <radius>0.039</radius>
+            <length>0.112</length>
           </cylinder>
         </geometry>
@@ -348,6 +360,6 @@
         <geometry>
           <cylinder>
-            <radius>r_thruster</radius>
-            <length>l_thruster</length>
+            <radius>0.039</radius>
+            <length>0.112</length>
           </cylinder>
         </geometry>
@@ -412,5 +424,5 @@
         <pose>0 0 0 0 -0 0</pose>
       </inertial>
-      <pose>-p_up_x -p_up_y p_z 0 -0 0</pose>
+      <pose>-0.539 -0.961 -1.5 0 -0 0</pose>
       <gravity>1</gravity>
       <self_collide>0</self_collide>
@@ -421,6 +433,6 @@
         <geometry>
           <cylinder>
-            <radius>r_thruster</radius>
-            <length>l_thruster</length>
+            <radius>0.039</radius>
+            <length>0.112</length>
           </cylinder>
         </geometry>
@@ -448,6 +460,6 @@
         <geometry>
           <cylinder>
-            <radius>r_thruster</radius>
-            <length>l_thruster</length>
+            <radius>0.039</radius>
+            <length>0.112</length>
           </cylinder>
         </geometry>
@@ -512,5 +524,5 @@
         <pose>0 0 0 0 -0 0</pose>
       </inertial>
-      <pose>p_up_x -p_up_y p_z 0 -0 0</pose>
+      <pose>0.539 -0.961 -1.5 0 -0 0</pose>
       <gravity>1</gravity>
       <self_collide>0</self_collide>
@@ -521,6 +533,6 @@
         <geometry>
           <cylinder>
-            <radius>r_thruster</radius>
-            <length>l_thruster</length>
+            <radius>0.039</radius>
+            <length>0.112</length>
           </cylinder>
         </geometry>
@@ -548,6 +560,6 @@
         <geometry>
           <cylinder>
-            <radius>r_thruster</radius>
-            <length>l_thruster</length>
+            <radius>0.039</radius>
+            <length>0.112</length>
           </cylinder>
         </geometry>
@@ -612,5 +624,5 @@
         <pose>0 0 0 0 -0 0</pose>
       </inertial>
-      <pose>-p_up_x p_side_y p_z 0 -0 0</pose>
+      <pose>-0.539 1.039 -1.5 0 -0 0</pose>
       <gravity>1</gravity>
       <self_collide>0</self_collide>
@@ -621,6 +633,6 @@
         <geometry>
           <cylinder>
-            <radius>r_thruster</radius>
-            <length>l_thruster</length>
+            <radius>0.039</radius>
+            <length>0.112</length>
           </cylinder>
         </geometry>
@@ -648,6 +660,6 @@
         <geometry>
           <cylinder>
-            <radius>r_thruster</radius>
-            <length>l_thruster</length>
+            <radius>0.039</radius>
+            <length>0.112</length>
           </cylinder>
         </geometry>
